File: kicad_files/Dart_launcher_robot_pcb/Dart_launcher_robot_pcb.kicad_sch (KiCad schematic)
At the start: 6 parts, among them J1 Conn_01x10_Pin, J11 Conn_01x10_Pin, J2 Conn_01x12_Pin, J40 Conn_01x02_Pin, J5 Conn_01x08_Pin, J6 Conn_01x08_Pin

Commit message: pcb design and changes to the pitch_yaw_launcher_code
Parts:
- removed J1, J11: Conn_01x10_Pin, Connector_PinHeader_2.54mm:PinHeader_1x10_P2.54mm_Vertical, symbol Connector:Conn_01x10_Pin
- removed J2: Conn_01x12_Pin, Connector_PinHeader_2.54mm:PinHeader_1x12_P2.54mm_Vertical, symbol Connector:Conn_01x12_Pin
- removed J40: Conn_01x02_Pin, Connector_PinHeader_2.54mm:PinHeader_1x02_P2.54mm_Vertical, symbol Connector:Conn_01x02_Pin
- removed J5, J6: Conn_01x08_Pin, Connector_PinHeader_2.54mm:PinHeader_1x08_P2.54mm_Vertical, symbol Connector:Conn_01x08_Pin
- added D1, D2, D4: LED, LED_SMD:LED_0805_2012Metric_Pad1.15x1.40mm_HandSolder, symbol Device:LED
- added H1, H2: MountingHole, MountingHole:MountingHole_3.2mm_M3, symbol Mechanical:MountingHole
- added J1, J11: 705430009, CONN_SDA-70543-xxxx_10_MOL, symbol Molex_705430009:705430009
- added J2: 705430011, CONN_SDA-70543-xxxx_12_MOL, symbol Molex_705430011:705430011
- added J23: 705430036, CONN_SDA-70543-xxxx_02_MOL, symbol Molex_705430036:705430036
- added J5, J6: 705430042, CONN_SDA-70543-xxxx_08_MOL, symbol Molex_705430042:705430042
- added R1, R2, R3: R_Small_US, Resistor_SMD:R_0603_1608Metric_Pad0.98x0.95mm_HandSolder, symbol Device:R_Small_US
Connections:
- net GND: now also J1.10, J23.1, R1.2, R2.2, R3.2
- net PA0: now also J5.1
- net PA1: now also J5.2
- net PA2: now also J5.3
- net PA3: now also J5.4
- net PA4: now also J11.8, J2.12
- net PA5: now also J1.8, J2.11
- net PB0: now also J11.4
- net PB1: now also J11.5
- net PC0: now also J11.6
- net PC1: now also J11.7, J2.7
- net PC2: now also J1.4
- net PC3: now also J1.5
- net PC4: now also J1.6
- net PC5: now also J1.7, J2.10
- net PD12: now also J6.1
- net PD13: now also J6.2
- net PD14: now also J6.3
- net PD15: now also J6.4
- net PE12: now also J11.3, J2.8
- net PE4: now also J11.2, J2.1
- net PE5: now also J1.2, J2.6
- net PE6: now also J1.3, J2.9
- net PF0: now also J11.1, J2.3
- net PF1: now also J1.1, J2.5
- net PF10: now also J1.9, J2.2
- net PH10: now also J6.5
- net PH11: now also J6.6
- net PH12: now also J6.7
- net PI0: now also J6.8
- net PI2: now also J5.8
- net PI5: now also J5.5
- net PI6: now also J5.6
- net PI7: now also J5.7
- net PI9: now also J11.9, J2.4
- net VCC_5V_U: now also D1.2 (A), J11.10, J23.2
- new net: D4.1 (K), R1.1
- new net: D1.1 (K), R2.1
- new net: D2.1 (K), R3.1
- new net 3V3: D2.2 (A)
- new net VCC_5V_ADJ: D4.2 (A)
